Commit message: Add files via upload

File: gazebo_sim_integration/gazebo_body_files/rover.urdf.xacro (robot description, xacro)
@@ -1,277 +1,283 @@
 <?xml version="1.0"?>
-<robot xmlns:xacro="http://www.ros.org/wiki/xacro" name="lunar_rover">
-    <xacro:property name="chassis_mass" value="40.0"/>
-    <xacro:property name="chassis_length" value="1.0"/>
-    <xacro:property name="chassis_width" value="0.6"/>
-    <xacro:property name="chassis_height" value="0.8"/> <xacro:property name="wheel_mass" value="5.0"/>
-    <xacro:property name="wheel_radius" value="0.2"/>
-    <xacro:property name="wheel_width" value="0.15"/>
-    <xacro:property name="moon_mu1" value="0.9"/>
-    <xacro:property name="moon_mu2" value="0.7"/>
-    <link name="base_link">
-        <visual>
-            <origin xyz="0 0 0" rpy="0 0 0"/>
-            <geometry>
-                <box size="${chassis_length} ${chassis_width} ${chassis_height}"/>
-            </geometry>
-        </visual>
-        <collision>
-            <origin xyz="0 0 0" rpy="0 0 0"/>
-            <geometry>
-                <box size="${chassis_length} ${chassis_width} ${chassis_height}"/>
-            </geometry>
-        </collision>
-        <inertial>
-            <mass value="${chassis_mass}"/>
-            <origin xyz="0 0 0" rpy="0 0 0"/>
-            <inertia ixx="1.0" ixy="0.0" ixz="0.0" iyy="1.0" iyz="0.0" izz="1.0"/>
-        </inertial>
+<robot xmlns:xacro="http://www.ros.org/wiki/xacro" name="alam_rover2">
+  <!-- Gazebo test rover body for moon-world side-by-side spawn -->
+  <!-- Expected folder: /root/ws/assets/custom/rover_body_2 -->
+  <xacro:property name="texture_root" value="/root/ws/assets/custom/rover_body_2/textures"/>
+  <xacro:property name="chassis_mass" value="55.0"/>
+  <xacro:property name="chassis_length" value="1.20"/>
+  <xacro:property name="chassis_width" value="0.78"/>
+  <xacro:property name="chassis_height" value="0.24"/>
+  <xacro:property name="chassis_clearance" value="0.03"/>
+  <xacro:property name="wheel_mass" value="4.0"/>
+  <xacro:property name="wheel_radius" value="0.18"/>
+  <xacro:property name="wheel_width" value="0.12"/>
+  <xacro:property name="wheel_y_offset" value="0.44"/>
+  <xacro:property name="wheel_z" value="0.0"/>
+  <xacro:property name="body_z" value="${wheel_radius + chassis_clearance + chassis_height/2.0}"/>
+  <xacro:property name="mast_z" value="${body_z + chassis_height/2.0 + 0.40}"/>
+  <xacro:property name="panel_z" value="${body_z + chassis_height/2.0 + 0.03}"/>
+  <xacro:property name="moon_mu1" value="1.10"/>
+  <xacro:property name="moon_mu2" value="0.95"/>
+  <!-- Base body -->
+  <link name="base_link">
+    <visual>
+      <origin xyz="0 0 ${body_z}" rpy="0 0 0"/>
+      <geometry>
+        <box size="${chassis_length} ${chassis_width} ${chassis_height}"/>
+      </geometry>
+    </visual>
+    <collision>
+      <origin xyz="0 0 ${body_z}" rpy="0 0 0"/>
+      <geometry>
+        <box size="${chassis_length} ${chassis_width} ${chassis_height}"/>
+      </geometry>
+    </collision>
+    <inertial>
+      <mass value="${chassis_mass}"/>
+      <origin xyz="0 0 ${body_z}" rpy="0 0 0"/>
+      <inertia ixx="3.5" ixy="0.0" ixz="0.0" iyy="8.0" iyz="0.0" izz="9.0"/>
+    </inertial>
+  </link>
+  <gazebo reference="base_link">
+    <self_collide>false</self_collide>
+    <visual>
+      <material>
+        <ambient>0.6 0.6 0.6 1.0</ambient>
+        <diffuse>0.6 0.6 0.6 1.0</diffuse>
+        <pbr>
+          <metal>
+            <albedo_map>file://${texture_root}/Silver/Poliigon_MetalSteelBrushed_7174_BaseColor.jpg</albedo_map>
+            <normal_map>file://${texture_root}/Silver/Poliigon_MetalSteelBrushed_7174_Normal.jpg</normal_map>
+            <roughness_map>file://${texture_root}/Silver/Poliigon_MetalSteelBrushed_7174_Roughness.jpg</roughness_map>
+            <metalness_map>file://${texture_root}/Silver/Poliigon_MetalSteelBrushed_7174_Metallic.jpg</metalness_map>
+            <ambient_occlusion_map>file://${texture_root}/Silver/Poliigon_MetalSteelBrushed_7174_AmbientOcclusion.jpg</ambient_occlusion_map>
+          </metal>
+        </pbr>
+      </material>
+    </visual>
+  </gazebo>
+  <!-- Mast -->
+  <link name="mast_link">
+    <visual>
+      <origin xyz="0 0 0.40" rpy="0 0 0"/>
+      <geometry>
+        <cylinder radius="0.04" length="0.80"/>
+      </geometry>
+    </visual>
+    <collision>
+      <origin xyz="0 0 0.40" rpy="0 0 0"/>
+      <geometry>
+        <cylinder radius="0.04" length="0.80"/>
+      </geometry>
+    </collision>
+    <inertial>
+      <mass value="1.5"/>
+      <origin xyz="0 0 0.40" rpy="0 0 0"/>
+      <inertia ixx="0.05" ixy="0.0" ixz="0.0" iyy="0.05" iyz="0.0" izz="0.005"/>
+    </inertial>
+  </link>
+  <joint name="mast_joint" type="fixed">
+    <parent link="base_link"/>
+    <child link="mast_link"/>
+    <origin xyz="-0.42 0 ${body_z + chassis_height/2.0}" rpy="0 0 0"/>
+  </joint>
+  <gazebo reference="mast_link">
+    <visual>
+      <material>
+        <ambient>0.35 0.35 0.35 1.0</ambient>
+        <diffuse>0.35 0.35 0.35 1.0</diffuse>
+        <pbr>
+          <metal>
+            <albedo_map>file://${texture_root}/Plastic/Poliigon_PlasticMoldDryBlast_7495_BaseColor.jpg</albedo_map>
+            <normal_map>file://${texture_root}/Plastic/Poliigon_PlasticMoldDryBlast_7495_Normal.jpg</normal_map>
+            <roughness_map>file://${texture_root}/Plastic/Poliigon_PlasticMoldDryBlast_7495_Roughness.jpg</roughness_map>
+            <metalness_map>file://${texture_root}/Plastic/Poliigon_PlasticMoldDryBlast_7495_Metallic.jpg</metalness_map>
+            <ambient_occlusion_map>file://${texture_root}/Plastic/Poliigon_PlasticMoldDryBlast_7495_AmbientOcclusion.jpg</ambient_occlusion_map>
+          </metal>
+        </pbr>
+      </material>
+    </visual>
+  </gazebo>
+  <!-- Simple temporary front arm and bucket -->
+  <link name="arm_link">
+    <visual>
+      <origin xyz="0.20 0 0" rpy="0 0 0"/>
+      <geometry>
+        <box size="0.40 0.08 0.05"/>
+      </geometry>
+    </visual>
+    <collision>
+      <origin xyz="0.20 0 0" rpy="0 0 0"/>
+      <geometry>
+        <box size="0.40 0.08 0.05"/>
+      </geometry>
+    </collision>
+    <inertial>
+      <mass value="2.0"/>
+      <origin xyz="0.20 0 0" rpy="0 0 0"/>
+      <inertia ixx="0.03" ixy="0.0" ixz="0.0" iyy="0.05" iyz="0.0" izz="0.05"/>
+    </inertial>
+  </link>
+  <joint name="arm_joint" type="revolute">
+    <parent link="base_link"/>
+    <child link="arm_link"/>
+    <origin xyz="${chassis_length/2.0 - 0.14} 0 ${body_z - 0.03}" rpy="0 0 0"/>
+    <axis xyz="0 1 0"/>
+    <limit lower="-0.50" upper="0.70" effort="60.0" velocity="0.8"/>
+  </joint>
+  <link name="bucket_link">
+    <visual>
+      <origin xyz="0 0 0" rpy="0 0 0"/>
+      <geometry>
+        <box size="0.18 0.34 0.14"/>
+      </geometry>
+    </visual>
+    <collision>
+      <origin xyz="0 0 0" rpy="0 0 0"/>
+      <geometry>
+        <box size="0.18 0.34 0.14"/>
+      </geometry>
+    </collision>
+    <inertial>
+      <mass value="2.5"/>
+      <origin xyz="0 0 0" rpy="0 0 0"/>
+      <inertia ixx="0.02" ixy="0.0" ixz="0.0" iyy="0.02" iyz="0.0" izz="0.02"/>
+    </inertial>
+  </link>
+  <joint name="bucket_joint" type="fixed">
+    <parent link="arm_link"/>
+    <child link="bucket_link"/>
+    <origin xyz="0.40 0 0" rpy="0 0 0"/>
+  </joint>
+  <gazebo reference="bucket_link">
+    <visual>
+      <material>
+        <ambient>0.55 0.45 0.10 1.0</ambient>
+        <diffuse>0.55 0.45 0.10 1.0</diffuse>
+        <pbr>
+          <metal>
+            <albedo_map>file://${texture_root}/Gold/Poliigon_MetalGoldPaint_7253_BaseColor.jpg</albedo_map>
+            <normal_map>file://${texture_root}/Gold/Poliigon_MetalGoldPaint_7253_Normal.jpg</normal_map>
+            <roughness_map>file://${texture_root}/Gold/Poliigon_MetalGoldPaint_7253_Roughness.jpg</roughness_map>
+            <metalness_map>file://${texture_root}/Gold/Poliigon_MetalGoldPaint_7253_Metallic.jpg</metalness_map>
+            <ambient_occlusion_map>file://${texture_root}/Gold/Poliigon_MetalGoldPaint_7253_AmbientOcclusion.jpg</ambient_occlusion_map>
+          </metal>
+        </pbr>
+      </material>
+    </visual>
+  </gazebo>
+  <!-- Solar panel -->
+  <link name="solar_panel_link">
+    <visual>
+      <origin xyz="0 0 0" rpy="0 0 0"/>
+      <geometry>
+        <box size="0.70 0.44 0.02"/>
+      </geometry>
+    </visual>
+    <collision>
+      <origin xyz="0 0 0" rpy="0 0 0"/>
+      <geometry>
+        <box size="0.70 0.44 0.02"/>
+      </geometry>
+    </collision>
+    <inertial>
+      <mass value="0.8"/>
+      <origin xyz="0 0 0" rpy="0 0 0"/>
+      <inertia ixx="0.01" ixy="0.0" ixz="0.0" iyy="0.02" iyz="0.0" izz="0.02"/>
+    </inertial>
+  </link>
+  <joint name="solar_panel_joint" type="fixed">
+    <parent link="base_link"/>
+    <child link="solar_panel_link"/>
+    <origin xyz="0 0 ${panel_z}" rpy="0 0 0"/>
+  </joint>
+  <gazebo reference="solar_panel_link">
+    <visual>
+      <material>
+        <ambient>0.20 0.20 0.25 1.0</ambient>
+        <diffuse>0.20 0.20 0.25 1.0</diffuse>
+        <pbr>
+          <metal>
+            <albedo_map>file://${texture_root}/Slate/Poliigon_SlateFloorTile_7657_BaseColor.jpg</albedo_map>
+            <normal_map>file://${texture_root}/Slate/Poliigon_SlateFloorTile_7657_Normal.jpg</normal_map>
+            <roughness_map>file://${texture_root}/Slate/Poliigon_SlateFloorTile_7657_Roughness.jpg</roughness_map>
+            <metalness_map>file://${texture_root}/Slate/Poliigon_SlateFloorTile_7657_Metallic.jpg</metalness_map>
+            <ambient_occlusion_map>file://${texture_root}/Slate/Poliigon_SlateFloorTile_7657_AmbientOcclusion.jpg</ambient_occlusion_map>
+          </metal>
+        </pbr>
+      </material>
+    </visual>
+  </gazebo>
+  <!-- Wheel macro -->
+  <xacro:macro name="rover_wheel" params="prefix x_offset y_offset">
+    <link name="${prefix}_wheel">
+      <visual>
+        <origin xyz="0 0 0" rpy="1.5708 0 0"/>
+        <geometry>
+          <cylinder radius="${wheel_radius}" length="${wheel_width}"/>
+        </geometry>
+      </visual>
+      <collision>
+        <origin xyz="0 0 0" rpy="1.5708 0 0"/>
+        <geometry>
+          <cylinder radius="${wheel_radius}" length="${wheel_width}"/>
+        </geometry>
+      </collision>
+      <inertial>
+        <mass value="${wheel_mass}"/>
+        <origin xyz="0 0 0" rpy="1.5708 0 0"/>
+        <inertia ixx="0.04" ixy="0.0" ixz="0.0" iyy="0.04" iyz="0.0" izz="0.04"/>
+      </inertial>
     </link>
-    <gazebo reference="base_link">
-        <visual>
-            <material>
-                <pbr>
-                    <metal>
-                        <albedo_map>file://textures/Poliigon_MetalSteelBrushed_7174_BaseColor.jpg</albedo_map>
-                        <normal_map>file://textures/Poliigon_MetalSteelBrushed_7174_Normal.jpg</normal_map>
-                        <roughness_map>file://textures/Poliigon_MetalSteelBrushed_7174_Roughness.jpg</roughness_map>
-                        <metalness_map>file://textures/Poliigon_MetalSteelBrushed_7174_Metallic.jpg</metalness_map>
-                        <ambient_occlusion_map>file://textures/Poliigon_MetalSteelBrushed_7174_AmbientOcclusion.jpg</ambient_occlusion_map>
-                    </metal>
-                </pbr>
-            </material>
-        </visual>
+    <joint name="${prefix}_wheel_joint" type="continuous">
+      <parent link="base_link"/>
+      <child link="${prefix}_wheel"/>
+      <origin xyz="${x_offset} ${y_offset} ${wheel_z}" rpy="0 0 0"/>
+      <axis xyz="0 1 0"/>
+    </joint>
+    <gazebo reference="${prefix}_wheel">
+      <mu1>${moon_mu1}</mu1>
+      <mu2>${moon_mu2}</mu2>
+      <self_collide>false</self_collide>
+      <visual>
+        <material>
+          <ambient>0.18 0.18 0.18 1.0</ambient>
+          <diffuse>0.18 0.18 0.18 1.0</diffuse>
+          <pbr>
+            <metal>
+              <albedo_map>file://${texture_root}/Ceramic/TilesCeramicHerringbone002_COL_2K.jpg</albedo_map>
+              <normal_map>file://${texture_root}/Ceramic/TilesCeramicHerringbone002_NRM_2K.jpg</normal_map>
+              <roughness_map>file://${texture_root}/Ceramic/TilesCeramicHerringbone002_GLOSS_2K.jpg</roughness_map>
+              <ambient_occlusion_map>file://${texture_root}/Ceramic/TilesCeramicHerringbone002_AO_2K.jpg</ambient_occlusion_map>
+            </metal>
+          </pbr>
+        </material>
+      </visual>
     </gazebo>
-    <link name="mast_link">
-        <visual>
-            <origin xyz="0 0 0.5" rpy="0 0 0"/>
-            <geometry>
-                <cylinder radius="0.05" length="1.0"/>
-            </geometry>
-        </visual>
-        <collision>
-            <origin xyz="0 0 0.5" rpy="0 0 0"/>
-            <geometry>
-                <cylinder radius="0.05" length="1.0"/>
-            </geometry>
-        </collision>
-        <inertial>
-            <mass value="2.0"/>
-            <origin xyz="0 0 0.5" rpy="0 0 0"/>
-            <inertia ixx="0.1" ixy="0.0" ixz="0.0" iyy="0.1" iyz="0.0" izz="0.01"/>
-        </inertial>
-    </link>
-    <joint name="mast_joint" type="fixed">
-        <parent link="base_link"/>
-        <child link="mast_link"/>
-        <origin xyz="-0.4 0 ${chassis_height/2}" rpy="0 0 0"/>
-    </joint>
-    <gazebo reference="mast_link">
-        <visual>
-            <material>
-                <pbr>
-                    <metal>
-                        <albedo_map>file://textures/Poliigon_PlasticMoldDryBlast_7495_BaseColor.jpg</albedo_map>
-                        <normal_map>file://textures/Poliigon_PlasticMoldDryBlast_7495_Normal.jpg</normal_map>
-                        <roughness_map>file://textures/Poliigon_PlasticMoldDryBlast_7495_Roughness.jpg</roughness_map>
-                        <metalness_map>file://textures/Poliigon_PlasticMoldDryBlast_7495_Metallic.jpg</metalness_map>
-                        <ambient_occlusion_map>file://textures/Poliigon_PlasticMoldDryBlast_7495_AmbientOcclusion.jpg</ambient_occlusion_map>
-                    </metal>
-                </pbr>
-            </material>
-        </visual>
-        <light type="spot" name="viper_headlight_left">
-            <pose>0.1 0.2 0.8 0 0 0</pose>
-            <diffuse>1 1 1 1</diffuse>
-            <specular>0.2 0.2 0.2 1</specular>
-            <attenuation>
-                <range>30</range>
-                <linear>0.01</linear>
-                <constant>0.2</constant>
-                <quadratic>0.001</quadratic>
-            </attenuation>
-            <spot>
-                <inner_angle>0.5</inner_angle>
-                <outer_angle>1.0</outer_angle>
-                <falloff>1.0</falloff>
-            </spot>
-            <cast_shadows>true</cast_shadows>
-        </light>
-    </gazebo>
-    <link name="arm_link">
-        <visual>
-            <origin xyz="0.2 0 0" rpy="0 0 0"/>
-            <geometry>
-                <box size="0.4 0.1 0.05"/>
-            </geometry>
-        </visual>
-        <collision>
-            <origin xyz="0.2 0 0" rpy="0 0 0"/>
-            <geometry>
-                <box size="0.4 0.1 0.05"/>
-            </geometry>
-        </collision>
-        <inertial>
-            <mass value="3.0"/>
-            <origin xyz="0.2 0 0" rpy="0 0 0"/>
-            <inertia ixx="0.1" ixy="0.0" ixz="0.0" iyy="0.1" iyz="0.0" izz="0.1"/>
-        </inertial>
-    </link>
-    <joint name="arm_joint" type="revolute">
-        <parent link="base_link"/>
-        <child link="arm_link"/>
-        <origin xyz="${chassis_length/2} 0 -0.2" rpy="0 0 0"/>
-        <axis xyz="0 1 0"/>
-        <limit lower="-0.5" upper="0.5" effort="100" velocity="1.0"/>
-    </joint>
-    <link name="bucket_link">
-        <visual>
-            <origin xyz="0 0 0" rpy="0 0 0"/>
-            <geometry>
-                <box size="0.2 0.6 0.3"/>
-            </geometry>
-        </visual>
-        <collision>
-            <origin xyz="0 0 0" rpy="0 0 0"/>
-            <geometry>
-                <box size="0.2 0.6 0.3"/>
-            </geometry>
-        </collision>
-        <inertial>
-            <mass value="5.0"/>
-            <origin xyz="0 0 0" rpy="0 0 0"/>
-            <inertia ixx="0.1" ixy="0.0" ixz="0.0" iyy="0.1" iyz="0.0" izz="0.1"/>
-        </inertial>
-    </link>
-    <joint name="bucket_joint" type="fixed">
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